Commit message: add laser plugin

File: urdf/IMU/IMU.gazebo.xacro (robot description, xacro)
@@ -4,6 +4,5 @@
     <gazebo reference="imu_link">
       <sensor type="imu" name="imu_sensor">
-        <plugin name="ignition::gazebo::systems::Imu" filename="libignition-gazebo-imu-system.so" >
-        </plugin>
+        <plugin name="ignition::gazebo::systems::Imu" filename="libignition-gazebo-imu-system.so" />
         <topic>/imu</topic>
         <origin xyz="0 0 0" rpy="0 0 0" />

File: urdf/laser/laser.gazebo.xacro (robot description, xacro)
@@ -2,9 +2,16 @@
 <robot xmlns:xacro="http://ros.org/wiki/xacro">
   <xacro:macro name="laser_gazebo">
+    <gazebo>
+      <plugin filename="libignition-gazebo-sensors-system.so"
+        name="ignition::gazebo::systems::Sensors">
+        <render_engine>ogre2</render_engine>
+      </plugin>
+    </gazebo>
     <gazebo reference="laser_scan">
-      <sensor type="ray" name="laser_scan_sensor">
-        <always_on>true</always_on>
+      <sensor name='gpu_lidar' type='gpu_lidar'>
+        <pose>0 0 0.1 0 0 0</pose>
+        <topic>/scan</topic>
         <update_rate>5</update_rate>
-        <visualize>false</visualize>
+        <gz_frame_id>laser_scan</gz_frame_id>
         <ray>
           <scan>
@@ -12,29 +19,17 @@
               <samples>360</samples>
               <resolution>1</resolution>
-              <!-- <min_angle>-2.35619449</min_angle>
-            <max_angle>2.35619449</max_angle> -->
-              <!-- <min_angle>0.0</min_angle>
-              <max_angle>6.28319</max_angle> -->
-              <min_angle>-3.14159274</min_angle>
-              <max_angle>3.14159274</max_angle>
+              <min_angle>-3.1415</min_angle>
+              <max_angle>3.1415</max_angle>
             </horizontal>
           </scan>
           <range>
-            <min>0.12</min>
-            <max>5</max>
+            <min>0.08</min>
+            <max>10.0</max>
             <resolution>0.01</resolution>
           </range>
-          <noise>
-            <type>gaussian</type>
-            <mean>0.0</mean>
-            <stddev>0.01</stddev>
-          </noise>
         </ray>
-        <!-- <plugin name="laser_controller" filename="libgazebo_ros_laser.so">
-          <topicName>/scan</topicName>
-          <frameName>laser_scan</frameName>
-        </plugin> -->
+        <always_on>true</always_on>
+        <visualize>true</visualize>
       </sensor>
-      <material>Gazebo/Red</material>
     </gazebo>
   </xacro:macro>

Commit message: small update on imu and laser urdf

File: urdf/IMU/IMU.gazebo.xacro (robot description, xacro)
@@ -2,14 +2,13 @@
 <robot xmlns:xacro="http://ros.org/wiki/xacro">
   <xacro:macro name="imu_gazebo_v0">
+    <gazebo>
+      <plugin name="ignition::gazebo::systems::Imu" filename="libignition-gazebo-imu-system.so" />
+    </gazebo>
     <gazebo reference="imu_link">
       <sensor type="imu" name="imu_sensor">
-        <plugin name="ignition::gazebo::systems::Imu" filename="libignition-gazebo-imu-system.so" />
         <topic>/imu</topic>
-        <origin xyz="0 0 0" rpy="0 0 0" />
         <update_rate>50</update_rate>
         <always_on>1</always_on>
         <visualize>1</visualize>
-        <imu>
-        </imu>
       </sensor>
     </gazebo>

File: urdf/laser/laser.gazebo.xacro (robot description, xacro)
@@ -10,5 +10,4 @@
     <gazebo reference="laser_scan">
       <sensor name='gpu_lidar' type='gpu_lidar'>
-        <pose>0 0 0.1 0 0 0</pose>
         <topic>/scan</topic>
         <update_rate>5</update_rate>
