Commit message: add camera to gazebo

File: urdf/3w_omni_robot.urdf.xacro (robot description, xacro)
@@ -10,6 +10,9 @@
   <xacro:include filename="$(find ros2_omni_robot_sim)/urdf/roller/roller.urdf.xacro" />   <!--roller-->
   <xacro:include filename="$(find ros2_omni_robot_sim)/urdf/IMU/IMU.urdf.xacro" />   <!--IMU-->
-  <xacro:include filename="$(find ros2_omni_robot_sim)/urdf/laser/laser.urdf.xacro" />   Laser
+  <xacro:include filename="$(find ros2_omni_robot_sim)/urdf/laser/laser.urdf.xacro" />   <!-- Laser -->
   <xacro:include filename="$(find ros2_omni_robot_sim)/urdf/camera_bracket/camera_bracket.urdf.xacro" />   <!--camera_bracket-->
+  <xacro:include filename="$(find ros2_omni_robot_sim)/urdf/gazebo_plugins.urdf.xacro" />   <!--Gazebo Plugins -->
+  <!-- ============ Gazebo Plugins ============== -->
+  <xacro:gazebo_plugins />
   <!-- =============== Link & Joint =============== -->
   <!-- Base -->

File: urdf/IMU/IMU.gazebo.xacro (robot description, xacro)
@@ -2,7 +2,4 @@
 <robot xmlns:xacro="http://ros.org/wiki/xacro">
   <xacro:macro name="imu_gazebo_v0">
-    <gazebo>
-      <plugin name="ignition::gazebo::systems::Imu" filename="libignition-gazebo-imu-system.so" />
-    </gazebo>
     <gazebo reference="imu_link">
       <sensor type="imu" name="imu_sensor">

File: urdf/camera/camera.gazebo.xacro (robot description, xacro)
@@ -2,41 +2,41 @@
 <robot xmlns:xacro="http://ros.org/wiki/xacro">
   <xacro:macro name="camera_gazebo_v0" params="prefix">
-	 <gazebo reference="${prefix}_camera_link">
-          <sensor type="camera" name="${prefix}">
-            <update_rate>10.0</update_rate>
-            <camera name="${prefix}_camera">
-              <pose>0 0 0 0 0 0</pose>
-              <horizontal_fov>1.3962634</horizontal_fov>
-              <image>
-                <width>640</width>
-                <height>480</height>
-                <format>R8G8B8</format>
-              </image>
-              <clip>
-               <near>0.02</near>
-               <far>300</far>
-              </clip>
-              <noise>
-                <type>gaussian</type>
-                <mean>0.0</mean>
-                <stddev>0.007</stddev>
-              </noise>
-            </camera>
-            <!-- <plugin name="camera_controller" filename="libgazebo_ros_camera.so">
-              <alwaysOn>true</alwaysOn>
-              <updateRate>0.0</updateRate>
-              <cameraName>${prefix}_camera</cameraName>
-              <imageTopicName>image_raw</imageTopicName>
-              <cameraInfoTopicName>camera_info</cameraInfoTopicName>
-              <frameName>${prefix}_link</frameName>
-              <hackBaseline>0.0</hackBaseline>
-              <distortionK1>0.0</distortionK1>
-              <distortionK2>0.0</distortionK2>
-              <distortionK3>0.0</distortionK3>
-              <distortionT1>0.0</distortionT1>
-              <distortionT2>0.0</distortionT2>
-            </plugin> -->
-          </sensor>
-        </gazebo>
+    <gazebo reference="${prefix}_camera_link">
+      <sensor type="depth" name="${prefix}_depth_camera">
+        <topic>depth</topic>
+        <update_rate>10.0</update_rate>
+        <camera name="${prefix}_camera">
+          <pose>0 0 0 0 0 0</pose>
+          <horizontal_fov>1.57</horizontal_fov>
+          <image>
+            <width>320</width>
+            <height>240</height>
+            <format>R8G8B8</format>
+          </image>
+          <clip>
+            <near>0.02</near>
+            <far>300</far>
+          </clip>
+          <noise>
+            <type>gaussian</type>
+            <mean>0.0</mean>
+            <stddev>0.007</stddev>
+          </noise>
+        </camera>
+      </sensor>
+      <sensor name="${prefix}_camera" type="camera">
+        <camera>
+          <horizontal_fov>1.57</horizontal_fov>
+          <image>
+            <width>640</width>
+            <height>480</height>
+          </image>
+        </camera>
+        <always_on>1</always_on>
+        <update_rate>30</update_rate>
+        <visualize>true</visualize>
+        <topic>camera</topic>
+      </sensor>
+    </gazebo>
   </xacro:macro>
 </robot>

File: urdf/camera/camera.urdf.xacro (robot description, xacro)
@@ -1,28 +1,28 @@
 <?xml version="1.0"?>
 <robot name="delirobo" xmlns:xacro="http://ros.org/wiki/xacro">
-  <xacro:include filename="$(find ros2_omni_robot_sim)/urdf/camera/camera.gazebo.xacro"/>
-  <xacro:macro name="camera_v0" params="prefix parent *joint_origin">
-	<joint name="${prefix}_camera_joint" type="fixed">
-	  <xacro:insert_block name="joint_origin"/>
-	  <parent link="${parent}"/>
-	  <child link="${prefix}_camera_link"/>
-	</joint>
-	<link name="${prefix}_camera_link">
-	  <visual>
-		<geometry>
-		  <mesh filename="package://ros2_omni_robot_sim/meshes/DAE/camera/camera.dae"/>
-		</geometry>
-	  </visual>
-	  <collision>
-		<geometry>
-		  <mesh filename="package://ros2_omni_robot_sim/meshes/STL/camera/camera.stl"/>
-		</geometry>
-	  </collision>
-	  <inertial>
-		<origin xyz="0 0 0"/>
-		<mass value="0.1"/>
-		<inertia ixx="0.00001" ixy="0" ixz="0" iyy="0.00001" iyz="0" izz="0.00001" />
-	  </inertial>
-	</link>
-  </xacro:macro>
+	<xacro:include filename="$(find ros2_omni_robot_sim)/urdf/camera/camera.gazebo.xacro" />
+	<xacro:macro name="camera_v0" params="prefix parent *joint_origin">
+		<joint name="${prefix}_camera_joint" type="fixed">
+			<xacro:insert_block name="joint_origin" />
+			<parent link="${parent}" />
+			<child link="${prefix}_camera_link" />
+		</joint>
+		<link name="${prefix}_camera_link">
+			<visual>
+				<geometry>
+					<mesh filename="package://ros2_omni_robot_sim/meshes/DAE/camera/camera.dae" />
+				</geometry>
+			</visual>
+			<collision>
+				<geometry>
+					<mesh filename="package://ros2_omni_robot_sim/meshes/STL/camera/camera.stl" />
+				</geometry>
+			</collision>
+			<inertial>
+				<origin xyz="0 0 0" />
+				<mass value="0.1" />
+				<inertia ixx="0.00001" ixy="0" ixz="0" iyy="0.00001" iyz="0" izz="0.00001" />
+			</inertial>
+		</link>
+	</xacro:macro>
 </robot>

File: urdf/laser/laser.gazebo.xacro (robot description, xacro)
@@ -2,10 +2,10 @@
 <robot xmlns:xacro="http://ros.org/wiki/xacro">
   <xacro:macro name="laser_gazebo">
-    <gazebo>
+    <!-- <gazebo>
       <plugin filename="libignition-gazebo-sensors-system.so"
         name="ignition::gazebo::systems::Sensors">
         <render_engine>ogre2</render_engine>
       </plugin>
-    </gazebo>
+    </gazebo> -->
     <gazebo reference="laser_scan">
       <sensor name='gpu_lidar' type='gpu_lidar'>

Commit message: add ros2_control

File: urdf/3w_omni_robot.urdf.xacro (robot description, xacro)
@@ -13,6 +13,5 @@
   <xacro:include filename="$(find ros2_omni_robot_sim)/urdf/camera_bracket/camera_bracket.urdf.xacro" />   <!--camera_bracket-->
   <xacro:include filename="$(find ros2_omni_robot_sim)/urdf/gazebo_plugins.urdf.xacro" />   <!--Gazebo Plugins -->
-  <!-- ============ Gazebo Plugins ============== -->
-  <xacro:gazebo_plugins />
+  <xacro:include filename="$(find ros2_omni_robot_sim)/urdf/ros2_control.urdf.xacro" />   <!-- Ros2 Control Plugins -->
   <!-- =============== Link & Joint =============== -->
   <!-- Base -->
@@ -22,4 +21,6 @@
   </xacro:base_v0>
   <!-- <xacro:base_v1 parent="base_footprint" xyz="0 0 0" rpy="0 0 ${-M_PI/2}" /> -->
+  <!-- Base -->
+  <xacro:base_gazebo_v0 />
   <!-- Base Layer -->
   <!-- <xacro:base_layer prefix="first" parent="base_footprint" xyz="0 0 0.125" rpy="0 0 ${M_PI/2}" /> -->
@@ -169,5 +170,5 @@
     <origin xyz="0 0 0.061" rpy="0 0.5236 0" />
   </xacro:camera_v0>
-  <!-- camera bracket-->
+  <!-- camera bracket -->
   <xacro:camera_bracket_v0 prefix="main" parent="base_link">
     <origin xyz="0 0 0.039" rpy="0 0 1.570796" />
@@ -176,16 +177,4 @@
   <!-- Laser -->
   <xacro:laser parent="first_base_layer_link" xyz="0 0 0.0065" rpy="0 0 0" />
-  <!-- ===============  Transmission =============== -->
-  <!-- <xacro:wheel_trans_v0 prefix="first" />
-  <xacro:wheel_trans_v0 prefix="second" />
-  <xacro:wheel_trans_v0 prefix="third" />
-  <xacro:camera_bracket_trans_v0 prefix="main" /> -->
-  <!-- =============== Gazebo =============== -->
-  <!-- <gazebo>
-    <plugin name="gazebo_ros_control" filename="libgazebo_ros_control.so">
-    </plugin>
-  </gazebo> -->
-  <!-- Base -->
-  <xacro:base_gazebo_v0 />
   <!-- Wheel -->
   <!-- <xacro:wheel_gazebo_v0 prefix="first" />

File: urdf/gazebo_plugins.urdf.xacro (robot description, xacro)
@@ -1,11 +1,13 @@
 <?xml version="1.0"?>
 <robot xmlns:xacro="http://ros.org/wiki/xacro">
-  <xacro:macro name="gazebo_plugins">
-    <gazebo>
-      <plugin filename="libignition-gazebo-sensors-system.so" name="ignition::gazebo::systems::Sensors">
-        <render_engine>ogre2</render_engine>
-      </plugin>
-      <plugin name="ignition::gazebo::systems::Imu" filename="libignition-gazebo-imu-system.so" />
-    </gazebo>
-  </xacro:macro>
+  <gazebo>
+    <plugin filename="libignition-gazebo-sensors-system.so"
+      name="ignition::gazebo::systems::Sensors">
+      <render_engine>ogre2</render_engine>
+    </plugin>
+    <plugin name="ignition::gazebo::systems::Imu" filename="libignition-gazebo-imu-system.so" />
+    <plugin filename="ign_ros2_control-system" name="ign_ros2_control::IgnitionROS2ControlPlugin">
+      <parameters>$(find ros2_omni_robot_sim)/config/controller_config.yaml</parameters>
+    </plugin>
+  </gazebo>
 </robot>
