Commit message: update urdf and controller_config of robot model 3w to make the wheel joint and link name identical as 3w_v2

File: urdf/3w/main.urdf.xacro (robot description, xacro)
@@ -28,135 +28,135 @@
   <!-- Wheel -->
   <!-- 1st wheel -->
-  <xacro:wheel_v0 prefix="first" parent="base_link">
+  <xacro:wheel_v0 suffix="1" parent="base_link">
     <origin xyz="0 0.088 -0.01" rpy="0 0 3.141593" />
     <axis xyz="0 1 0" />
   </xacro:wheel_v0>
-  <xacro:roller_v0 prefix="r1_F" parent="first_wheel_link">
+  <xacro:roller_v0 prefix="r1_F" parent="omni_wheel_link_1">
     <origin xyz="0 -0.006 0.024063" rpy="0 0 1.570796" />
     <axis xyz="0 1 0" />
   </xacro:roller_v0>
-  <xacro:roller_v0 prefix="r2_F" parent="first_wheel_link">
+  <xacro:roller_v0 prefix="r2_F" parent="omni_wheel_link_1">
     <origin xyz="-0.0228853 -0.006 0.0074359" rpy="-1.256637 0 1.570796" />
     <axis xyz="0 1 0" />
   </xacro:roller_v0>
-  <xacro:roller_v0 prefix="r3_F" parent="first_wheel_link">
+  <xacro:roller_v0 prefix="r3_F" parent="omni_wheel_link_1">
     <origin xyz="-0.0141439 -0.006 -0.0194674" rpy="-2.513274 0 1.570796" />
     <axis xyz="0 1 0" />
   </xacro:roller_v0>
-  <xacro:roller_v0 prefix="r4_F" parent="first_wheel_link">
+  <xacro:roller_v0 prefix="r4_F" parent="omni_wheel_link_1">
     <origin xyz="0.0141439 -0.006 -0.0194674" rpy="-3.769911 0 1.570796" />
     <axis xyz="0 1 0" />
   </xacro:roller_v0>
-  <xacro:roller_v0 prefix="r5_F" parent="first_wheel_link">
+  <xacro:roller_v0 prefix="r5_F" parent="omni_wheel_link_1">
     <origin xyz="0.0228853 -0.006 0.0074359" rpy="-5.026548 0 1.570796" />
     <axis xyz="0 1 0" />
   </xacro:roller_v0>
-  <xacro:roller_v0 prefix="r6_F" parent="first_wheel_link">
+  <xacro:roller_v0 prefix="r6_F" parent="omni_wheel_link_1">
     <origin xyz="0 0.006 -0.024063" rpy="0 0 1.570796" />
     <axis xyz="0 1 0" />
   </xacro:roller_v0>
-  <xacro:roller_v0 prefix="r7_F" parent="first_wheel_link">
+  <xacro:roller_v0 prefix="r7_F" parent="omni_wheel_link_1">
     <origin xyz="0.0228853 0.006 -0.0074359" rpy="-1.256637 0 1.570796" />
     <axis xyz="0 1 0" />
   </xacro:roller_v0>
-  <xacro:roller_v0 prefix="r8_F" parent="first_wheel_link">
+  <xacro:roller_v0 prefix="r8_F" parent="omni_wheel_link_1">
     <origin xyz="0.0141439 0.006 0.0194674" rpy="-2.513274 0 1.570796" />
     <axis xyz="0 1 0" />
   </xacro:roller_v0>
-  <xacro:roller_v0 prefix="r9_F" parent="first_wheel_link">
+  <xacro:roller_v0 prefix="r9_F" parent="omni_wheel_link_1">
     <origin xyz="-0.0141439 0.006 0.0194674" rpy="-3.769911 0 1.570796" />
     <axis xyz="0 1 0" />
   </xacro:roller_v0>
-  <xacro:roller_v0 prefix="r10_F" parent="first_wheel_link">
+  <xacro:roller_v0 prefix="r10_F" parent="omni_wheel_link_1">
     <origin xyz="-0.0228853 0.006 -0.0074359" rpy="-5.026548 0 1.570796" />
     <axis xyz="0 1 0" />
   </xacro:roller_v0>
   <!-- 2nd wheel -->
-  <xacro:wheel_v0 prefix="second" parent="base_link">
+  <xacro:wheel_v0 suffix="2" parent="base_link">
     <origin xyz="-0.0762 -0.044 -0.01" rpy="0 0 5.235988" />
     <axis xyz="0 1 0" />
   </xacro:wheel_v0>
-  <xacro:roller_v0 prefix="r1_S" parent="second_wheel_link">
+  <xacro:roller_v0 prefix="r1_S" parent="omni_wheel_link_2">
     <origin xyz="0 -0.006 0.024063" rpy="0 0 1.570796" />
     <axis xyz="0 1 0" />
   </xacro:roller_v0>
-  <xacro:roller_v0 prefix="r2_S" parent="second_wheel_link">
+  <xacro:roller_v0 prefix="r2_S" parent="omni_wheel_link_2">
     <origin xyz="-0.0228853 -0.006 0.0074359" rpy="-1.256637 0 1.570796" />
     <axis xyz="0 1 0" />
   </xacro:roller_v0>
-  <xacro:roller_v0 prefix="r3_S" parent="second_wheel_link">
+  <xacro:roller_v0 prefix="r3_S" parent="omni_wheel_link_2">
     <origin xyz="-0.0141439 -0.006 -0.0194674" rpy="-2.513274 0 1.570796" />
     <axis xyz="0 1 0" />
   </xacro:roller_v0>
-  <xacro:roller_v0 prefix="r4_S" parent="second_wheel_link">
+  <xacro:roller_v0 prefix="r4_S" parent="omni_wheel_link_2">
     <origin xyz="0.0141439 -0.006 -0.0194674" rpy="-3.769911 0 1.570796" />
     <axis xyz="0 1 0" />
   </xacro:roller_v0>
-  <xacro:roller_v0 prefix="r5_S" parent="second_wheel_link">
+  <xacro:roller_v0 prefix="r5_S" parent="omni_wheel_link_2">
     <origin xyz="0.0228853 -0.006 0.0074359" rpy="-5.026548 0 1.570796" />
     <axis xyz="0 1 0" />
   </xacro:roller_v0>
-  <xacro:roller_v0 prefix="r6_S" parent="second_wheel_link">
+  <xacro:roller_v0 prefix="r6_S" parent="omni_wheel_link_2">
     <origin xyz="0 0.006 -0.024063" rpy="0 0 1.570796" />
     <axis xyz="0 1 0" />
   </xacro:roller_v0>
-  <xacro:roller_v0 prefix="r7_S" parent="second_wheel_link">
+  <xacro:roller_v0 prefix="r7_S" parent="omni_wheel_link_2">
     <origin xyz="0.0228853 0.006 -0.0074359" rpy="-1.256637 0 1.570796" />
     <axis xyz="0 1 0" />
   </xacro:roller_v0>
-  <xacro:roller_v0 prefix="r8_S" parent="second_wheel_link">
+  <xacro:roller_v0 prefix="r8_S" parent="omni_wheel_link_2">
     <origin xyz="0.0141439 0.006 0.0194674" rpy="-2.513274 0 1.570796" />
     <axis xyz="0 1 0" />
   </xacro:roller_v0>
-  <xacro:roller_v0 prefix="r9_S" parent="second_wheel_link">
+  <xacro:roller_v0 prefix="r9_S" parent="omni_wheel_link_2">
     <origin xyz="-0.0141439 0.006 0.0194674" rpy="-3.769911 0 1.570796" />
     <axis xyz="0 1 0" />
   </xacro:roller_v0>
-  <xacro:roller_v0 prefix="r10_S" parent="second_wheel_link">
+  <xacro:roller_v0 prefix="r10_S" parent="omni_wheel_link_2">
     <origin xyz="-0.0228853 0.006 -0.0074359" rpy="-5.026548 0 1.570796" />
     <axis xyz="0 1 0" />
   </xacro:roller_v0>
   <!-- 3rd wheel -->
-  <xacro:wheel_v0 prefix="third" parent="base_link">
+  <xacro:wheel_v0 suffix="3" parent="base_link">
     <origin xyz="0.0762 -0.044 -0.01" rpy="0 0 1.047197" />
     <axis xyz="0 1 0" />
   </xacro:wheel_v0>
-  <xacro:roller_v0 prefix="r1_T" parent="third_wheel_link">
+  <xacro:roller_v0 prefix="r1_T" parent="omni_wheel_link_3">
     <origin xyz="0 -0.006 0.024063" rpy="0 0 1.570796" />
     <axis xyz="0 1 0" />
   </xacro:roller_v0>
-  <xacro:roller_v0 prefix="r2_T" parent="third_wheel_link">
+  <xacro:roller_v0 prefix="r2_T" parent="omni_wheel_link_3">
     <origin xyz="-0.0228853 -0.006 0.0074359" rpy="-1.256637 0 1.570796" />
     <axis xyz="0 1 0" />
   </xacro:roller_v0>
-  <xacro:roller_v0 prefix="r3_T" parent="third_wheel_link">
+  <xacro:roller_v0 prefix="r3_T" parent="omni_wheel_link_3">
     <origin xyz="-0.0141439 -0.006 -0.0194674" rpy="-2.513274 0 1.570796" />
     <axis xyz="0 1 0" />
   </xacro:roller_v0>
-  <xacro:roller_v0 prefix="r4_T" parent="third_wheel_link">
+  <xacro:roller_v0 prefix="r4_T" parent="omni_wheel_link_3">
     <origin xyz="0.0141439 -0.006 -0.0194674" rpy="-3.769911 0 1.570796" />
     <axis xyz="0 1 0" />
   </xacro:roller_v0>
-  <xacro:roller_v0 prefix="r5_T" parent="third_wheel_link">
+  <xacro:roller_v0 prefix="r5_T" parent="omni_wheel_link_3">
     <origin xyz="0.0228853 -0.006 0.0074359" rpy="-5.026548 0 1.570796" />
     <axis xyz="0 1 0" />
   </xacro:roller_v0>
-  <xacro:roller_v0 prefix="r6_T" parent="third_wheel_link">
+  <xacro:roller_v0 prefix="r6_T" parent="omni_wheel_link_3">
     <origin xyz="0 0.006 -0.024063" rpy="0 0 1.570796" />
     <axis xyz="0 1 0" />
   </xacro:roller_v0>
-  <xacro:roller_v0 prefix="r7_T" parent="third_wheel_link">
+  <xacro:roller_v0 prefix="r7_T" parent="omni_wheel_link_3">
     <origin xyz="0.0228853 0.006 -0.0074359" rpy="-1.256637 0 1.570796" />
     <axis xyz="0 1 0" />
   </xacro:roller_v0>
-  <xacro:roller_v0 prefix="r8_T" parent="third_wheel_link">
+  <xacro:roller_v0 prefix="r8_T" parent="omni_wheel_link_3">
     <origin xyz="0.0141439 0.006 0.0194674" rpy="-2.513274 0 1.570796" />
     <axis xyz="0 1 0" />
   </xacro:roller_v0>
-  <xacro:roller_v0 prefix="r9_T" parent="third_wheel_link">
+  <xacro:roller_v0 prefix="r9_T" parent="omni_wheel_link_3">
     <origin xyz="-0.0141439 0.006 0.0194674" rpy="-3.769911 0 1.570796" />
     <axis xyz="0 1 0" />
   </xacro:roller_v0>
-  <xacro:roller_v0 prefix="r10_T" parent="third_wheel_link">
+  <xacro:roller_v0 prefix="r10_T" parent="omni_wheel_link_3">
     <origin xyz="-0.0228853 0.006 -0.0074359" rpy="-5.026548 0 1.570796" />
     <axis xyz="0 1 0" />

File: urdf/3w/omni_wheel/omni_wheel.gazebo.xacro (robot description, xacro)
@@ -1,6 +1,6 @@
 <?xml version="1.0"?>
 <robot xmlns:xacro="http://ros.org/wiki/xacro">
-  <xacro:macro name="wheel_gazebo_v0" params="prefix">
-	<gazebo reference="${prefix}_wheel_link">
+  <xacro:macro name="wheel_gazebo_v0" params="suffix">
+	<gazebo reference="omni_wheel_link_${suffix}">
 	  <selfCollide>false</selfCollide>
       <mu1 value="0.8" />

File: urdf/3w/omni_wheel/omni_wheel.urdf.xacro (robot description, xacro)
@@ -1,15 +1,15 @@
 <?xml version="1.0"?>
 <robot xmlns:xacro="http://ros.org/wiki/xacro">
-  <xacro:include filename="$(find ros2_omni_robot_sim)/urdf/3w/omni_wheel/omni_wheel.transmission.xacro"/>
-  <xacro:include filename="$(find ros2_omni_robot_sim)/urdf/3w/omni_wheel/omni_wheel.gazebo.xacro"/>
-  <xacro:macro name="wheel_v0" params="prefix parent *joint_origin *joint_axis">
-	<joint name="${prefix}_wheel_joint" type="continuous">
+  <!-- <xacro:include filename="$(find ros2_omni_robot_sim)/urdf/3w/omni_wheel/omni_wheel.transmission.xacro"/>
+  <xacro:include filename="$(find ros2_omni_robot_sim)/urdf/3w/omni_wheel/omni_wheel.gazebo.xacro"/> -->
+  <xacro:macro name="wheel_v0" params="suffix parent *joint_origin *joint_axis">
+	<joint name="omni_wheel_joint_${suffix}" type="continuous">
 	  <xacro:insert_block name="joint_origin"/>
 	  <parent link="${parent}"/>
-	  <child link="${prefix}_wheel_link"/>
+	  <child link="omni_wheel_link_${suffix}"/>
           <limit effort="100" velocity="100"/>
 	  <xacro:insert_block name="joint_axis"/>
 	</joint>
-	<link name="${prefix}_wheel_link">
+	<link name="omni_wheel_link_${suffix}">
 	  <visual>
 		<geometry>

File: urdf/3w/ros2_control.urdf.xacro (robot description, xacro)
@@ -5,5 +5,5 @@
             <plugin>ign_ros2_control/IgnitionSystem</plugin>
         </hardware>
-        <joint name="first_wheel_joint">
+        <joint name="omni_wheel_joint_1">
             <command_interface name="velocity">
                 <param name="min">-10</param>
@@ -13,5 +13,5 @@
             <state_interface name="velocity" />
         </joint>
-        <joint name="second_wheel_joint">
+        <joint name="omni_wheel_joint_2">
             <command_interface name="velocity">
                 <param name="min">-10</param>
@@ -21,5 +21,5 @@
             <state_interface name="velocity" />
         </joint>
-        <joint name="third_wheel_joint">
+        <joint name="omni_wheel_joint_3">
             <command_interface name="velocity">
                 <param name="min">-10</param>
