Commit message: fix issue for 4w, 5w, and 6w robot

File: urdf/6w/base_link.urdf.xacro (robot description, xacro)
@@ -11,7 +11,7 @@
           <mesh filename="package://ros2_omni_robot_sim/meshes/6w/base_link.stl" />
         </geometry>
-        <material name="base_color">
+        <!-- <material name="base_color">
           <color rgba="0.34 0.55 0.949 1" />
-        </material>
+        </material> -->
       </visual>
       <collision>
