Commit message: update urdf and meshes

File: urdf/3w_v2/base_link.urdf.xacro (robot description, xacro)
@@ -9,9 +9,9 @@
       <visual>
         <geometry>
-          <mesh filename="package://ros2_omni_robot_sim/meshes/3w_v2/base_link.stl" />
+          <mesh filename="package://ros2_omni_robot_sim/meshes/3w_v2/base_link.dae" />
         </geometry>
-        <material name="base_color">
+        <!-- <material name="base_color">
           <color rgba="0.34 0.55 0.949 1" />
-        </material>
+        </material> -->
       </visual>
       <collision>

File: urdf/3w_v2/lidar.urdf.xacro (robot description, xacro)
@@ -7,6 +7,6 @@
           <cylinder radius="0.02" length="0.02" />
         </geometry>
-        <material name="blue">
-          <color rgba="0 0 1 1" />
+        <material name="red">
+          <color rgba="0.4 0 0.1 1" />
         </material>
       </visual>

File: urdf/4w/base_link.urdf.xacro (robot description, xacro)
@@ -9,9 +9,9 @@
       <visual>
         <geometry>
-          <mesh filename="package://ros2_omni_robot_sim/meshes/4w/base_link.stl" />
+          <mesh filename="package://ros2_omni_robot_sim/meshes/4w/base_link.dae" />
         </geometry>
-        <material name="base_color">
+        <!-- <material name="base_color">
           <color rgba="0.34 0.55 0.949 1" />
-        </material>
+        </material> -->
       </visual>
       <collision>

File: urdf/4w/lidar.urdf.xacro (robot description, xacro)
@@ -8,5 +8,5 @@
         </geometry>
         <material name="blue">
-          <color rgba="0 0 1 1" />
+          <color rgba="0.1 0 0.35 1" />
         </material>
       </visual>

File: urdf/5w/base_link.urdf.xacro (robot description, xacro)
@@ -9,9 +9,9 @@
       <visual>
         <geometry>
-          <mesh filename="package://ros2_omni_robot_sim/meshes/5w/base_link.stl" />
+          <mesh filename="package://ros2_omni_robot_sim/meshes/5w/base_link.dae" />
         </geometry>
-        <material name="base_color">
+        <!-- <material name="base_color">
           <color rgba="0.34 0.55 0.949 1" />
-        </material>
+        </material> -->
       </visual>
       <collision>

File: urdf/5w/lidar.urdf.xacro (robot description, xacro)
@@ -7,6 +7,6 @@
           <cylinder radius="0.02" length="0.02" />
         </geometry>
-        <material name="blue">
-          <color rgba="0 0 1 1" />
+        <material name="yellow">
+          <color rgba="0.35 0.35 0.01 1" />
         </material>
       </visual>

File: urdf/6w/base_link.urdf.xacro (robot description, xacro)
@@ -9,5 +9,5 @@
       <visual>
         <geometry>
-          <mesh filename="package://ros2_omni_robot_sim/meshes/6w/base_link.stl" />
+          <mesh filename="package://ros2_omni_robot_sim/meshes/6w/base_link.dae" />
         </geometry>
         <!-- <material name="base_color">

File: urdf/6w/lidar.urdf.xacro (robot description, xacro)
@@ -7,6 +7,6 @@
           <cylinder radius="0.02" length="0.02" />
         </geometry>
-        <material name="blue">
-          <color rgba="0 0 1 1" />
+        <material name="green">
+          <color rgba="0 0.25 0.05 1" />
         </material>
       </visual>
